Commit message: final commit

File: ex01/robot_gazebo_sim/urdf/robot.gazebo.xacro (robot description, xacro)
@@ -1,4 +1,38 @@
 <?xml version="1.0"?>
 <robot xmlns:xacro="http://www.ros.org/wiki/xacro">
+  <gazebo>
+    <plugin filename="gz-sim-imu-system" name="gz::sim::systems::Imu"/>
+  </gazebo>
+  <gazebo reference="imu_link">
+    <sensor name="imu_sensor" type="imu">
+      <always_on>true</always_on>
+      <update_rate>100</update_rate>
+      <visualize>true</visualize>
+      <topic>/imu</topic>
+      <pose>0 0 0 0 0 0</pose>
+      <imu>
+        <angular_velocity>
+          <x>0.0</x>
+          <y>0.0</y>
+          <z>0.0</z>
+        </angular_velocity>
+        <linear_acceleration>
+          <x>0.0</x>
+          <y>0.0</y>
+          <z>0.0</z>
+        </linear_acceleration>
+        <noise type="gaussian">
+          <rate>
+            <mean>0.0</mean>
+            <stddev>0.0002</stddev>
+          </rate>
+          <accel>
+            <mean>0.0</mean>
+            <stddev>0.002</stddev>
+          </accel>
+        </noise>
+      </imu>
+    </sensor>
+  </gazebo>
   <gazebo>
     <plugin filename="libgz-sim-joint-state-publisher-system.so" name="gz::sim::systems::JointStatePublisher">
@@ -28,5 +62,5 @@
       <visualize>true</visualize>
       <topic>/scan</topic>
-      <ray> <!-- для gpu_lidar в Gazebo Harmonic ray тоже поддерживается -->
+      <ray>
         <scan>
           <horizontal>
@@ -38,5 +72,4 @@
         </scan>
         <range>
-          <!-- НЕ ноль, иначе near clip = 0 и Ogre падает -->
           <min>0.1</min>
           <max>20.0</max>
@@ -44,4 +77,34 @@
         </range>
       </ray>
+    </sensor>
+  </gazebo>
+  <gazebo reference="tower">
+    <sensor name="depth_camera" type="depth_camera">
+      <update_rate>6</update_rate>
+      <always_on>1</always_on>
+      <visualize>true</visualize>
+      <topic>/depth_camera/image</topic>
+      <pose>0.1 0 0.4 0 0 0</pose>
+      <camera>
+        <horizontal_fov>1.51843645</horizontal_fov>
+        <image>
+          <width>848</width>
+          <height>480</height>
+          <format>R_FLOAT32</format>
+        </image>
+        <clip>
+          <near>0.1</near>
+          <far>10</far>
+        </clip>
+        <lens>
+          <intrinsics>
+            <fx>421.61578369140625</fx>
+            <fy>421.61578369140625</fy>
+            <cx>422.2854309082031</cx>
+            <cy>236.57237243652344</cy>
+            <s>0</s>
+          </intrinsics>
+        </lens>
+      </camera>
     </sensor>
   </gazebo>

File: ex01/robot_gazebo_sim/urdf/robot.urdf.xacro (robot description, xacro)
@@ -1,5 +1,4 @@
 <?xml version="1.0"?>
 <robot xmlns:xacro="http://www.ros.org/wiki/xacro" name="tank_robot">
-  <!-- Параметры -->
   <xacro:property name="base_length" value="0.7"/>
   <xacro:property name="base_width" value="0.5"/>
@@ -9,16 +8,12 @@
   <xacro:property name="wheel_offset_y" value="0.225"/>
   <xacro:property name="wheel_offset_x" value="0.2"/>
-  <!-- Башня -->
   <xacro:property name="tower_radius" value="0.2"/>
   <xacro:property name="tower_height" value="0.25"/>
   <xacro:property name="tower_offset_x" value="0.1"/>
-  <!-- Дуло -->
   <xacro:property name="barrel_radius" value="0.025"/>
   <xacro:property name="barrel_length" value="0.6"/>
-  <!-- Материалы (зелёный танк) -->
   <material name="army_green"><color rgba="0.2 0.6 0.2 1"/></material>
   <material name="dark_green"><color rgba="0.1 0.4 0.1 1"/></material>
   <material name="black"><color rgba="0.05 0.05 0.05 1"/></material>
-  <!-- Корпус (зелёный танк) -->
   <link name="base_link">
     <visual>
@@ -36,5 +31,4 @@
     </inertial>
   </link>
-  <!-- Макрос колеса -->
   <xacro:macro name="wheel" params="name x y">
     <link name="${name}">
@@ -60,10 +54,8 @@
     </joint>
   </xacro:macro>
-  <!-- 4 колеса -->
   <xacro:wheel name="front_left_wheel"  x="${wheel_offset_x}"  y="${wheel_offset_y}"/>
   <xacro:wheel name="front_right_wheel" x="${wheel_offset_x}"  y="-${wheel_offset_y}"/>
   <xacro:wheel name="rear_left_wheel"   x="-${wheel_offset_x}" y="${wheel_offset_y}"/>
   <xacro:wheel name="rear_right_wheel"  x="-${wheel_offset_x}" y="-${wheel_offset_y}"/>
-  <!-- Башня (вращающаяся) -->
   <link name="tower">
     <visual>
@@ -87,5 +79,4 @@
     <axis xyz="0 1 0"/>
   </joint>
-  <!-- Дуло (на башне) -->
   <link name="barrel">
     <visual>
@@ -108,4 +99,10 @@
     <origin xyz="0 0 0" rpy="0 0 0"/>
   </joint>
+  <link name="imu_link"/>
+  <joint name="imu_joint" type="fixed">
+      <parent link="base_link"/>
+      <child link="imu_link"/>
+      <origin xyz="0.1 0 0.15" rpy="0 0 0"/>
+  </joint>
   <!-- Gazebo плагины -->
   <xacro:include filename="robot.gazebo.xacro"/>

File: ex02/robot_gazebo_sim/urdf/robot.gazebo.xacro (robot description, xacro)
@@ -1,4 +1,38 @@
 <?xml version="1.0"?>
 <robot xmlns:xacro="http://www.ros.org/wiki/xacro">
+  <gazebo>
+    <plugin filename="gz-sim-imu-system" name="gz::sim::systems::Imu"/>
+  </gazebo>
+  <gazebo reference="imu_link">
+    <sensor name="imu_sensor" type="imu">
+      <always_on>true</always_on>
+      <update_rate>100</update_rate>
+      <visualize>true</visualize>
+      <topic>/imu</topic>
+      <pose>0 0 0 0 0 0</pose>
+      <imu>
+        <angular_velocity>
+          <x>0.0</x>
+          <y>0.0</y>
+          <z>0.0</z>
+        </angular_velocity>
+        <linear_acceleration>
+          <x>0.0</x>
+          <y>0.0</y>
+          <z>0.0</z>
+        </linear_acceleration>
+        <noise type="gaussian">
+          <rate>
+            <mean>0.0</mean>
+            <stddev>0.0002</stddev>
+          </rate>
+          <accel>
+            <mean>0.0</mean>
+            <stddev>0.002</stddev>
+          </accel>
+        </noise>
+      </imu>
+    </sensor>
+  </gazebo>
   <gazebo>
     <plugin filename="libgz-sim-joint-state-publisher-system.so" name="gz::sim::systems::JointStatePublisher">
@@ -28,5 +62,5 @@
       <visualize>true</visualize>
       <topic>/scan</topic>
-      <ray> <!-- для gpu_lidar в Gazebo Harmonic ray тоже поддерживается -->
+      <ray>
         <scan>
           <horizontal>
@@ -38,5 +72,4 @@
         </scan>
         <range>
-          <!-- НЕ ноль, иначе near clip = 0 и Ogre падает -->
           <min>0.1</min>
           <max>20.0</max>

File: ex03/robot_gazebo_sim/urdf/robot.gazebo.xacro (robot description, xacro)
@@ -1,4 +1,38 @@
 <?xml version="1.0"?>
 <robot xmlns:xacro="http://www.ros.org/wiki/xacro">
+  <gazebo>
+    <plugin filename="gz-sim-imu-system" name="gz::sim::systems::Imu"/>
+  </gazebo>
+  <gazebo reference="imu_link">
+    <sensor name="imu_sensor" type="imu">
+      <always_on>true</always_on>
+      <update_rate>100</update_rate>
+      <visualize>true</visualize>
+      <topic>/imu</topic>
+      <pose>0 0 0 0 0 0</pose>
+      <imu>
+        <angular_velocity>
+          <x>0.0</x>
+          <y>0.0</y>
+          <z>0.0</z>
+        </angular_velocity>
+        <linear_acceleration>
+          <x>0.0</x>
+          <y>0.0</y>
+          <z>0.0</z>
+        </linear_acceleration>
+        <noise type="gaussian">
+          <rate>
+            <mean>0.0</mean>
+            <stddev>0.0002</stddev>
+          </rate>
+          <accel>
+            <mean>0.0</mean>
+            <stddev>0.002</stddev>
+          </accel>
+        </noise>
+      </imu>
+    </sensor>
+  </gazebo>
   <gazebo>
     <plugin filename="libgz-sim-joint-state-publisher-system.so" name="gz::sim::systems::JointStatePublisher">
@@ -28,5 +62,5 @@
       <visualize>true</visualize>
       <topic>/scan</topic>
-      <ray> <!-- для gpu_lidar в Gazebo Harmonic ray тоже поддерживается -->
+      <ray>
         <scan>
           <horizontal>
@@ -38,5 +72,4 @@
         </scan>
         <range>
-          <!-- НЕ ноль, иначе near clip = 0 и Ogre падает -->
           <min>0.1</min>
           <max>20.0</max>
@@ -76,25 +109,4 @@
     </sensor>
   </gazebo>
-    <!-- IMU на корпусе робота -->
-  <gazebo reference="base_link">
-    <sensor name="imu_sensor" type="imu">
-      <always_on>true</always_on>
-      <update_rate>100</update_rate>
-      <visualize>true</visualize>
-      <topic>/imu</topic>
-      <imu>
-        <angular_velocity>
-          <x>0.0</x>
-          <y>0.0</y>
-          <z>0.0</z>
-        </angular_velocity>
-        <linear_acceleration>
-          <x>0.0</x>
-          <y>0.0</y>
-          <z>0.0</z>
-        </linear_acceleration>
-      </imu>
-    </sensor>
-  </gazebo>
   <!-- Трение для колёс -->
   <gazebo reference="front_left_wheel">
